Commit message: add dooby_simulation final version

File: ROS/ros2_ws/src/dooby_simulation/src/description/dooby_simulation.urdf (robot description, URDF)
Before this commit: robot dooby_bot, 4 links, 3 joints
Links:
- added link camera_depth_frame
Joints:
- added joint camera_depth_joint: type fixed, parent camera_link, child camera_depth_frame, origin xyz=0 0 0 rpy=${-pi/2} 0 ${-pi/2}
